File: build/FM_DRUM_MACHINE/FM_DRUM_MACHINE.kicad_sch (KiCad schematic)
At the start: 218 parts, among them SW1 STEP1, SW10 STEP10, SW11 STEP11, SW12 STEP12, SW13 STEP13, SW14 STEP14, SW15 STEP15, SW16 STEP16, SW17 KICK_TRIG, SW18 SNARE_TRIG, SW19 CHAT_TRIG, SW2 STEP2, SW20 OHAT_TRIG, SW21 LOTOM_TRIG, SW22 HITOM_TRIG, SW23 PLAY/PAUSE, SW24 RECORD, SW25 SELECT, SW3 STEP3, SW4 STEP4, SW5 STEP5, SW6 STEP6, SW7 STEP7, SW8 STEP8, SW9 STEP9, U1 6N138, U2 TL072, U3 TL072, U4 TL074, U5 MAX7221xNG

Commit message: v0.2
- Further Schematic Modifications
Parts:
- removed B10k1: HiPass Cutoff, symbol Device:R_Potentiometer
- removed C1, C10, C11, C12, C13, C14, C15, C16, C17, C18, C19, C2, C20, C21, C22, C23, C24, C25, C26, C3, C4, C5, C6, C7, C8, C9: C, Capacitor_THT:C_Disc_D7.5mm_W2.5mm_P5.00mm, symbol Device:C
- removed C37: 47nF, Capacitor_THT:C_Disc_D7.5mm_W2.5mm_P5.00mm, symbol Device:C
- removed C38, C39, C40, C41: 10uF, symbol Device:C_Polarized_US
- removed Multiplexer1, Multiplexer2: CD74HC4067, MODULE, symbol CD74HC4067:CD74HC4067
- removed R53, R54, R55, R56, R57, R58, R59, R60: 10k, symbol Device:R
- removed R61, R62, R63, R64: 1k, symbol Device:R
- removed unit 3 of U2
- removed U4: TL074, symbol Amplifier_Operational:TL074
- removed cHatDecay, cHatFmFreq, cHatPitch, cHatTimbre, hiTomDecay, hiTomFmFreq, hiTomPitch, hiTomPunch, kickFmFreq, kickPitch, kickPunch, loTomDecay, loTomFmFreq, loTomPitch, loTomPunch, oHatDecay, oHatFmFreq, oHatPitch, oHatTimbre, snareDecay, snareFmFreq, snareNoiseBlend, snarePitch, snareSnap, snareTimbre: R_Potentiometer, PCM_4ms_Potentiometer:Pot_9mm_Knurl_NoDet, symbol Device:R_Potentiometer
- added A1, A2: GY-PCM5102, symbol gy-pcm5102:GY-PCM5102
- added C1, C2: 100uF, Capacitor_THT:CP_Radial_D5.0mm_P2.00mm, symbol Device:C_Polarized_US
- added C44, C45, C46, C47, C48, C49, C50, C51, C52, C53, C54, C55, C56, C57, C58, C59, C60, C61, C62, C63, C64, C65, C66, C67, C68: 10nF, PCM_4ms_Capacitor:C_Disc_P5.08mm, symbol Device:C
- added C69, C70, C71, C72, C73: 10uF, PCM_4ms_Capacitor:C_Disc_P5.08mm, symbol Device:C
- added D54: 1N914BWS, DIYSynthMNL:D_4148_BigPads, symbol PCM_4ms_Diode:1N914BWS
- added J1: 12V Centre +ve, Connector_BarrelJack:BarrelJack_SwitchcraftConxall_RAPC10U_Horizontal, symbol Connector:Jack-DC
- added Q1: BC547, Package_TO_SOT_THT:TO-92L_Inline, symbol Transistor_BJT:BC547
- added Q2: BC557, Package_TO_SOT_THT:TO-92_Inline, symbol Transistor_BJT:BC557
- added R70, R71: 100k, symbol Device:R
- added R72: 1k, symbol Device:R
- added RV10: SNARE_TIMBRE, PCM_4ms_Potentiometer:Pot_9mm_Knurl_NoDet, symbol Device:R_Potentiometer
- added RV11: CHAT_DECAY, PCM_4ms_Potentiometer:Pot_9mm_Knurl_NoDet, symbol Device:R_Potentiometer
- added RV12: CHAT_TIMBRE, PCM_4ms_Potentiometer:Pot_9mm_Knurl_NoDet, symbol Device:R_Potentiometer
- added RV13: CHAT_PITCH, PCM_4ms_Potentiometer:Pot_9mm_Knurl_NoDet, symbol Device:R_Potentiometer
- added RV14: CHAT_FMFREQ, PCM_4ms_Potentiometer:Pot_9mm_Knurl_NoDet, symbol Device:R_Potentiometer
- added RV15: LOTOM_DECAY, PCM_4ms_Potentiometer:Pot_9mm_Knurl_NoDet, symbol Device:R_Potentiometer
- added RV16: LOTOM_PUNCH, PCM_4ms_Potentiometer:Pot_9mm_Knurl_NoDet, symbol Device:R_Potentiometer
- added RV17: LOTOM_PITCH, PCM_4ms_Potentiometer:Pot_9mm_Knurl_NoDet, symbol Device:R_Potentiometer
- added RV18: LOTOM_FMFREQ, PCM_4ms_Potentiometer:Pot_9mm_Knurl_NoDet, symbol Device:R_Potentiometer
- added RV19: HITOM_DECAY, PCM_4ms_Potentiometer:Pot_9mm_Knurl_NoDet, symbol Device:R_Potentiometer
- added RV20: HITOM_PUNCH, PCM_4ms_Potentiometer:Pot_9mm_Knurl_NoDet, symbol Device:R_Potentiometer
- added RV21: HITOM_PITCH, PCM_4ms_Potentiometer:Pot_9mm_Knurl_NoDet, symbol Device:R_Potentiometer
- added RV22: HITOM_FMFREQ, PCM_4ms_Potentiometer:Pot_9mm_Knurl_NoDet, symbol Device:R_Potentiometer
- added RV23: OHAT_DECAY, PCM_4ms_Potentiometer:Pot_9mm_Knurl_NoDet, symbol Device:R_Potentiometer
- added RV24: OHAT_TIMBRE, PCM_4ms_Potentiometer:Pot_9mm_Knurl_NoDet, symbol Device:R_Potentiometer
- added RV25: OHAT_PITCH, PCM_4ms_Potentiometer:Pot_9mm_Knurl_NoDet, symbol Device:R_Potentiometer
- added RV26: OHAT_FMFREQ, PCM_4ms_Potentiometer:Pot_9mm_Knurl_NoDet, symbol Device:R_Potentiometer
- added RV3: KICK_PITCH, PCM_4ms_Potentiometer:Pot_9mm_Knurl_NoDet, symbol Device:R_Potentiometer
- added RV4: KICK_PUNCH, PCM_4ms_Potentiometer:Pot_9mm_Knurl_NoDet, symbol Device:R_Potentiometer
- added RV5: KICK_FMFREQ, PCM_4ms_Potentiometer:Pot_9mm_Knurl_NoDet, symbol Device:R_Potentiometer
- added RV6: SNARE_DECAY, PCM_4ms_Potentiometer:Pot_9mm_Knurl_NoDet, symbol Device:R_Potentiometer
- added RV7: SNARE_SNAP, PCM_4ms_Potentiometer:Pot_9mm_Knurl_NoDet, symbol Device:R_Potentiometer
- added RV8: SNARE_PITCH, PCM_4ms_Potentiometer:Pot_9mm_Knurl_NoDet, symbol Device:R_Potentiometer
- added RV9: SNARE_FM, PCM_4ms_Potentiometer:Pot_9mm_Knurl_NoDet, symbol Device:R_Potentiometer
- added U10: TL072, 4ms_Package_SSOP:TSSOP-8_4.4x3mm_Pitch0.65mm, symbol PCM_4ms_IC:TL072
- added unit 2 of U3
- added unit 3 of U3
- added U6, U7: CD74HC4067M, Package_SO:SOIC-24W_7.5x15.4mm_P1.27mm, symbol 74xx:CD74HC4067M
- added U8: AMS1117-5.0, Package_TO_SOT_SMD:SOT-223-3_TabPin2, symbol Regulator_Linear:AMS1117-5.0
- added U9: AMS1117-3.3, Package_TO_SOT_SMD:SOT-223-3_TabPin2, symbol Regulator_Linear:AMS1117-3.3
- C27, C43: value 10uF -> 10nF
- RV1: renamed from kickDecay; value R_Potentiometer -> KICK_DECAY
Connections:
- net 3.3V: now also RV1.3, A1.13 (XSMT), A1.6 (VIN), A2.13 (XSMT), A2.6 (VIN), C72.2, RV10.3, RV11.3, RV12.3, RV13.3, RV14.3, RV15.3, RV16.3, RV17.3, RV18.3, RV19.3, RV20.3, RV21.3, RV22.3, RV23.3, RV24.3, RV25.3, RV26.3, RV3.3, RV4.3, RV5.3, RV6.3, RV7.3, RV8.3, RV9.3, U9.2 (VO); no longer Nano.30 (VIN), Teensy4.0.31 (3V3)
- net 5V: now also Nano.30 (VIN), R10.2, R8.2, Teensy4.0.33 (VIN), U1.8 (VCC), C70.2, C71.2, U6.24 (VCC), U7.24 (VCC), U8.2 (VO), U9.3 (VI)
- net 5v: no longer R10.2, R8.2, Teensy4.0.33 (VIN), U1.8 (VCC)
- net CHAT_TRIG OUT: no longer Teensy4.0.4 (2_OUT2)
- net GND: now also A1.12 (FMT), A1.14 (DEMP), A1.15 (FLT), A1.5 (GND), A2.12 (FMT), A2.14 (DEMP), A2.15 (FLT), A2.5 (GND), C2.2, C44.2, C45.2, C46.2, C47.2, C48.2, C49.2, C50.2, C51.2, C52.2, C53.2, C54.2, C55.2, C56.2, C57.2, C58.2, C59.2, C60.2, C61.2, C62.2, C63.2, C64.2, C65.2, C66.2, C67.2, C68.2, C69.1, C70.1, C71.1, C72.1, C73.1, Q2.1 (C), R71.2, RV10.1, RV11.1, RV12.1, RV13.1, RV14.1, RV15.1, RV16.1, RV17.1, RV18.1, RV19.1, RV20.1, RV21.1, RV22.1, RV23.1, RV24.1, RV25.1, RV26.1, RV3.1, RV4.1, RV5.1, RV6.1, RV7.1, RV8.1, RV9.1, U3.4 (V-), U6.12 (GND), U6.15 (~{E}), U7.12 (GND), U7.15 (~{E}), U8.1 (GND), U9.1 (GND)
- net HITOM_TRIG OUT: no longer Teensy4.0.7 (5_IN2)
- net KICK_TRIG OUT: no longer Teensy4.0.2 (0_RX1_CRX2_CS1)
- net LOTOM_TRIG OUT: no longer Teensy4.0.6 (4_BCLK2)
- net MIDI OUT: now also Teensy4.0.2 (0_RX1_CRX2_CS1)
- net OHAT_TRIG OUT: no longer Teensy4.0.5 (3_LRCLK2)
- net SNARE_TRIG OUT: no longer Teensy4.0.3 (1_TX1_CTX2_MISO1)
- net A1LCK: now reaches Teensy4.0.27 (20_A6_TX5_LRCLK1)
- net A1LCK: now also A1.4 (LCK), A2.4 (LCK)
- net A1BCK: now reaches Teensy4.0.28 (21_A7_RX5_BCLK1)
- net A1BCK: now also A1.2 (BCK), A2.2 (BCK)
- net A1SCK: now reaches Teensy4.0.30 (23_A9_CRX1_MCLK1)
- net A1SCK: now also A1.1 (SCK), A2.1 (SCK)
- net A1DIN: now reaches Teensy4.0.9 (7_RX2_OUT1A)
- net A1DIN: now also A1.3 (DIN), A2.3 (DIN)
- net Mult1S0: no longer names the net of Teensy4.0.11 (9_OUT1C)
- net Mult1S1: no longer names the net of Teensy4.0.12 (10_CS_MQSR)
- net Mult1S2: no longer names the net of Teensy4.0.13 (11_MOSI_CTX1)
- net Mult1S3: no longer names the net of Teensy4.0.14 (12_MISO_MQSL)
- net Mult2S0: no longer names the net of Teensy4.0.23 (16_A2_RX4_SCL1)
- net Mult2S1: no longer names the net of Teensy4.0.24 (17_A3_TX4_SDA1)
- net Mult2S2: no longer names the net of Teensy4.0.25 (18_A4_SDA0)
- net Mult2S3: no longer names the net of Teensy4.0.26 (19_A5_SCL0)
- net Multiplexer1 Sig Out renamed U6SIG
- net U6SIG: now also U6.1 (COM)
- net Multiplexer2 Sig Out renamed U7SIG
- net U7SIG: now also U7.1 (COM)
- net kickDecay renamed KICK_DECAY
- net KICK_DECAY: now also C44.1, U6.9 (I0)
- new net: C1.2, C2.1, Q1.3 (E), Q2.3 (E), R72.2, U10.2 (-), U3.5 (+)
- new net: C69.2, D54.1 (K), U8.3 (VI)
- new net: Q1.2 (B), Q2.2 (B), R72.1, U10.1
- new net: C73.2, R70.2, R71.1, U10.3 (+)
- new net 12V: C1.1, D54.2 (A), J1.2, Q1.1 (C), R70.1, U3.8 (V+)
- new net AGND: A1.10 (AGND), A1.8 (AGND), A2.10 (AGND), A2.8 (AGND)
- new net CHAT_DECAY: C53.1, RV11.2, U6.22 (I9)
- new net CHAT_FMFREQ: C56.1, RV14.2, U6.19 (I12)
- new net CHAT_PITCH: C55.1, RV13.2, U6.21 (I10)
- new net CHAT_TIMBRE: C54.1, RV12.2, U6.20 (I11)
- new net HATS_OUT: A2.7 (LOUT)
- new net HITOM_DECAY: C61.1, RV19.2, U7.4 (I5)
- new net HITOM_FMFREQ: C64.1, RV22.2, U7.23 (I8)
- new net HITOM_PITCH: C63.1, RV21.2, U7.3 (I6)
- new net HITOM_PUNCH: C62.1, RV20.2, U7.2 (I7)
- new net KICK_FMFREQ: C47.1, RV5.2, U6.6 (I3)
- new net KICK_OUT: A1.7 (LOUT)
- new net KICK_PITCH: C45.1, RV3.2, U6.8 (I1)
- new net KICK_PUNCH: C46.1, RV4.2, U6.7 (I2)
- new net LOTOM_DECAY: C57.1, RV15.2, U7.8 (I1)
- new net LOTOM_FMFREQ: C60.1, RV18.2, U7.5 (I4)
- new net LOTOM_PITCH: C59.1, RV17.2, U7.7 (I2)
- new net LOTOM_PUNCH: C58.1, RV16.2, U7.6 (I3)
- new net OHAT_DECAY: C65.1, RV23.2, U6.18 (I13)
- new net OHAT_FMFREQ: C68.1, RV26.2, U7.9 (I0)
- new net OHAT_PITCH: C67.1, RV25.2, U6.17 (I14)
- new net OHAT_TIMBRE: C66.1, RV24.2, U6.16 (I15)
- new net SNARE_DECAY: C48.1, RV6.2, U6.5 (I4)
- new net SNARE_FM: C51.1, RV9.2, U6.2 (I7)
- new net SNARE_OUT: A1.9 (ROUT)
- new net SNARE_PITCH: C50.1, RV8.2, U6.4 (I5)
- new net SNARE_PUNCH: C49.1, RV7.2, U6.3 (I6)
- new net SNARE_TIMBRE: C52.1, RV10.2, U6.23 (I8)
- new net TOMS_OUT: A2.9 (ROUT)
- new net U6S0: U6.10 (S0)
- new net U6S1: U6.11 (S1)
- new net U6S2: U6.14 (S2)
- new net U6S3: U6.13 (S3)
- new net U7S0: U7.10 (S0)
- new net U7S1: U7.11 (S1)
- new net U7S2: U7.14 (S2)
- new net U7S3: U7.13 (S3)
- new net VGND: U3.6 (-), U3.7
Other:
- note added: "CHAT"
- note added: "DACS"
- note added: "FM DRUMS"
- note added: "HI TOM"
- note added: "INPUT POWER"
- note added: "KICK"
- note added: "LO TOM"
- note added: "MULTIPLEXERS"
- note added: "OHAT"
- note added: "SNARE"
- note added: "TEENSY"
- note removed: "CLOSED HAT Digital Pot Controls"
- note removed: "HI TOM Digital Pot Controls"
- note removed: "INDIVIDUAL OUTPUTS"
- note removed: "KICK Digital Pot Controls"
- note removed: "LO TOM Digital Pot Controls"
- note removed: "MULTIPLEXERS - TEENSY"
- note removed: "OPEN HAT Digital Pot Controls"
- note removed: "Op-Amp Power"
- note removed: "SNARE Digital Pot Controls"
- note removed: "SNARE FILTER STAGE"
- moved on the sheet: B100k, B10k, BC547, C27, C28, C29, C30, C31, C32, C33, C34, C35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

Commit message: v0.3
- Circuit schematic update
Parts:
- removed B100k: R_Potentiometer_Dual, symbol Device:R_Potentiometer_Dual
- removed B10k: HiPass Cutoff, symbol Device:R_Potentiometer
- removed BC547 (x2): NPN, symbol Simulation_SPICE:NPN
- removed C28, C32, C34, C35, C42: 10uF, symbol Device:C_Polarized_US
- removed C29, C30, C31: 100nF, Capacitor_THT:C_Disc_D7.5mm_W2.5mm_P5.00mm, symbol Device:C
- removed C33: 33nF, Capacitor_THT:C_Disc_D7.5mm_W2.5mm_P5.00mm, symbol Device:C
- removed C36: 47nF, Capacitor_THT:C_Disc_D7.5mm_W2.5mm_P5.00mm, symbol Device:C
- removed D3, D4: Random Diode, symbol PCM_4ms_Diode:D_Generic
- removed Drive: 20k, symbol Device:R_Potentiometer
- removed FilterBypass: SW_DPDT_x2, symbol Switch:SW_DPDT_x2
- removed R29: 47k, symbol Device:R
- removed R30, R36: 220k, symbol Device:R
- removed R31, R34, R35: 10k, symbol Device:R
- removed R32: 4k7, symbol Device:R
- removed R33, R37: 1k, symbol Device:R
- removed U2: TL072, symbol Amplifier_Operational:TL072
- added C3: 10uF, Capacitor_THT:CP_Radial_D5.0mm_P2.00mm, symbol Device:C_Polarized_US
- added C74, C76, C78, C81: 1uF, PCM_4ms_Capacitor:C_Disc_P5.08mm, symbol Device:C
- added C75, C77, C79, C80: 10nF, PCM_4ms_Capacitor:C_Disc_P5.08mm, symbol Device:C
- added C82: 10uF, PCM_4ms_Capacitor:C_Disc_P5.08mm, symbol Device:C
- added C83, C84, C85, C86, C87: 10Uf, PCM_4ms_Capacitor:C_Disc_P5.08mm, symbol Device:C
- added Ch5: 20k, symbol Device:R_Potentiometer
- added Ch6: 1k, symbol Device:R_Potentiometer
- added D3, D4, D55, D56, D57, D58, D59, D60, D61, D62, D63, D64, D65, D66, D67: 1N4148, Diode_THT:D_DO-35_SOD27_P5.08mm_Vertical_KathodeUp, symbol Diode:1N4148
- added J2: KICK_BUFFEREDOUT, audioConnectors_Edit:Jack_3.5mm_CUI_SJ1-3525N_Horizontal_edit, symbol Connector_Audio:AudioJack2
- added J3: SNARE_BUFFEREDOUT, audioConnectors_Edit:Jack_3.5mm_CUI_SJ1-3525N_Horizontal_edit, symbol Connector_Audio:AudioJack2
- added J4: HATS_BUFFEREDOUT, audioConnectors_Edit:Jack_3.5mm_CUI_SJ1-3525N_Horizontal_edit, symbol Connector_Audio:AudioJack2
- added J5: TOMS_BUFFEREDOUT, audioConnectors_Edit:Jack_3.5mm_CUI_SJ1-3525N_Horizontal_edit, symbol Connector_Audio:AudioJack2
- added J6: LINE_OUT, symbol Connector_Audio:AudioJack2
- added R53, R56, R60, R73: 200k, symbol Device:R
- added R54, R61, R75, R77, R78, R80, R81, R83, R84, R85, R86, R87: 100k, symbol Device:R
- added R55, R62: 33k, symbol Device:R
- added R57, R63: 10k, symbol Device:R
- added R58, R64: 6k8, symbol Device:R
- added R59, R74: 1M, symbol Device:R
- added R76, R79: 14k, symbol Device:R
- added R82: 1k, symbol Device:R
- added R88: 20k, symbol Device:R
- added R89: 4k7, symbol Device:R
- added R91: 100R, symbol Device:R
- added R92, R93, R94, R95, R96, R97, R98, R99: 220R, symbol Device:R
- added RV27, RV28: 100k, symbol Device:R_Potentiometer_Dual_Separate
- added RV29: R_Potentiometer, DIYSynthMNL:Potentiometer_RV09_BigPads, symbol Device:R_Potentiometer
- added RV30: A100k, DIYSynthMNL:Potentiometer_RV09_BigPads, symbol Device:R_Potentiometer
- added RV31: 20k, DIYSynthMNL:Potentiometer_RV09_BigPads, symbol Device:R_Potentiometer
- added RV32: 100k, DIYSynthMNL:Potentiometer_RV09_BigPads, symbol Device:R_Potentiometer
- added SW26, SW27: SW_DPDT_x2, PCM_4ms_Switch:Switch_Toggle_DPDT_SubMini, symbol Switch:SW_DPDT_x2
- added TRIM1, TRIM2: TrimPot_T73YEt_100k, DIYSynthMNL:Potentiometer_Bourns_3296W_Vertical_BigPads, symbol PCM_4ms_Potentiometer:TrimPot_T73YEt_100k
- added unit 3 of U10
- added unit 2 of U10
- added U11: TL074, DIYSynthMNL:DIP-14_W7.62mm_LongPads, symbol Amplifier_Operational:TL074
- added U12: TL072, 4ms_Package_SSOP:TSSOP-8_4.4x3mm_Pitch0.65mm, symbol PCM_4ms_IC:TL072
- added U13, U14, U4: TL074, symbol Amplifier_Operational:TL074
- added U2: TL072, Package_DIP:DIP-8_W7.62mm, symbol PCM_4ms_IC:TL072
- R49, R50: value 100k -> 10k
- R51: value 1k -> 22k
- R52: value 27k -> 1k
- U3: footprint 4ms_Package_SSOP:TSSOP-8_4.4x3mm_Pitch0.65mm -> Package_DIP:DIP-8_W7.62mm
Connections:
- net FILTERED KICK OUT is gone; now on net KICK_OUT: Ch1.3
- net FILTERED SNARE OUT is gone; now on net SNARE_OUT: Ch2.3
- net HATS OUT is gone; now on net HATS_OUT: Ch3.3
- net TOMS OUT is gone; now on net TOMS_OUT: Ch4.3
- net 12V: now also R49.2, R88.1, U10.8 (V+), U11.4 (V+), U12.8 (V+), U13.4 (V+), U14.4 (V+), U2.8 (V+), U4.4 (V+)
- net GND: now also R50.1, Ch6.1, J6.S, R96.2, R97.2, R98.2, R99.2, U10.4 (V-), U11.11 (V-), U12.4 (V-), U13.11 (V-), U14.11 (V-), U2.4 (V-), U4.11 (V-); no longer R52.1
- net U6S0: now also Teensy4.0.11 (9_OUT1C)
- net U6S1: now also Teensy4.0.12 (10_CS_MQSR)
- net U6S2: now also Teensy4.0.13 (11_MOSI_CTX1)
- net U6S3: now also Teensy4.0.14 (12_MISO_MQSL)
- net U7S0: now also Teensy4.0.23 (16_A2_RX4_SCL1)
- net U7S1: now also Teensy4.0.24 (17_A3_TX4_SDA1)
- net U7S2: now also Teensy4.0.25 (18_A4_SDA0)
- net U7S3: now also Teensy4.0.26 (19_A5_SCL0)
- net VGND: now also R52.1, C80.1, C82.1, R53.2, R55.1, R56.2, R58.2, R59.2, R60.2, R62.1, R64.2, R73.2, R74.2, R76.1, R79.1, R83.1, R87.1, R89.1, RV27.1, RV29.1, RV30.3, RV31.1, TRIM1.1 (Left), U13.3 (+)
- net at R45.2, R46.1: now also U2.6 (-)
- net at R49.1: now also R50.2, U3.3 (+), C3.1; no longer R46.2
- net KICKBUFFER_IN: now reaches Ch1.2, R38.1
- net KICKBUFFER_IN: now also U14.3 (+)
- net at R38.2, R39.2, R40.2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: now also U2.2 (-)
- net HATSBUFFER_IN: now reaches Ch3.2, R40.1
- net HATSBUFFER_IN: now also U14.10 (+)
- net at R44.2, R45.1: now also U2.1
- net TOMSBUFFER_IN: now reaches Ch4.2, R41.1
- net TOMSBUFFER_IN: now also U14.12 (+)
- net SOFTCLIP_OUT: now reaches R51.1, U3.1
- net SOFTCLIP_OUT: now also C83.1, D4.2 (A), D55.1 (K); no longer R50.2
- net at R47.1, R48.2: now also U2.5 (+)
- net at R42.1, R43.2: now also U2.3 (+)
- net SNAREBUFFER_IN: now reaches Ch2.2, R39.1
- net SNAREBUFFER_IN: now also U14.5 (+)
- removed net AGND: A1.10 (AGND), A1.8 (AGND), A2.10 (AGND), A2.8 (AGND)
- net DRUM SUM OUT: no longer names the net of R51.2
- net DRUM SUM OUT: now also U3.2 (-), Ch5.3, D3.1 (K), D56.2 (A)
- new net: SW26.1 (A), SW26.4 (A)
- new net: D59.2 (A), D65.2 (A), D66.1 (K), R81.1, R82.2
- new net: R80.1, R81.2, U13.2 (-)
- new net: D62.1 (K), R80.2, U13.1
- new net: D61.1 (K), D62.2 (A)
- new net: C78.2, R60.1, R61.1
- new net: R61.2, R62.2, U4.3 (+)
- new net: J6.T, R91.1
- new net: Ch6.3, R91.2
- new net: R89.2, RV32.1, RV32.2
- new net: C82.2, R86.1, RV32.3, TRIM2.1 (Left), TRIM2.2 (Center), U13.13 (-)
- new net: R86.2, R87.2, U13.10 (+)
- new net: J4.T, R94.1, R98.1
- new net: R78.1, R79.2, U10.6 (-)
- new net: R57.2, R58.1, U11.13 (-)
- new net: C80.2, RV28.5, RV28.6, U4.10 (+)
- new net: C75.1, U11.1, U11.2 (-)
- new net: C75.2, RV27.5, RV27.6, U11.10 (+)
- new net: C79.1, R63.1, U4.14
- new net: R63.2, R64.1, U4.13 (-)
- new net: R88.2, RV31.3
- new net: SW27.1 (A), SW27.4 (A)
- new net: J3.T, R93.1, R97.1
- new net: R85.1, RV31.2
- new net: R84.1, R85.2, U13.9 (-)
- new net: D3.2 (A), D4.1 (K)
- new net: C83.2, Ch6.2
- new net: RV27.4, U11.6 (-), U11.7
- new net: C84.1, U14.1, U14.2 (-)
- new net: C87.1, U14.13 (-), U14.14
- new net: D58.2 (A), D59.1 (K)
- new net: C77.1, R57.1, U11.14
- new net: C77.2, RV27.2, RV27.3, U11.5 (+)
- new net: D67.1 (K), TRIM2.3 (Right)
- new net: D67.2 (A), U13.14
- new net: C74.2, R53.1, R54.1
- new net: J5.T, R95.1, R99.1
- new net: R84.2, RV30.1, U13.8
- new net: RV30.2, U13.5 (+)
- new net: R54.2, R55.2, U11.3 (+)
- new net: D63.1 (K), D66.2 (A), R83.2, U13.6 (-)
- new net: D63.2 (A), D64.1 (K)
- new net: D55.2 (A), D56.1 (K)
- new net: D60.1 (K), D61.2 (A)
- new net: D57.1 (K), D60.2 (A), R77.2, U10.5 (+)
- new net: TRIM1.2 (Center), U11.12 (+)
- new net: C76.1, TRIM1.3 (Right), U11.8, U11.9 (-)
- new net: R75.2, R76.2, U12.3 (+)
- new net: RV29.2, U4.12 (+)
- new net: C81.1, RV29.3, U4.8, U4.9 (-)
- new net: D64.2 (A), D65.1 (K)
- new net: J2.T, R92.1, R96.1
- new net: C84.2, R92.2
- new net: C86.2, R94.2
- new net: D57.2 (A), D58.1 (K)
- new net: R82.1, U13.7
- new net: C85.1, U14.6 (-), U14.7
- new net: C85.2, R93.2
- new net: C86.1, U14.8, U14.9 (-)
- new net: C87.2, R95.2
- new net: RV28.1, U4.1, U4.2 (-)
- new net: C79.2, RV28.2, RV28.3, U4.5 (+)
- new net: RV28.4, U4.6 (-), U4.7
- new net: Ch5.1, Ch5.2, R52.2
- new net: R77.1, U12.1, U12.2 (-)
- new net AGND_HATS: A2.8 (AGND), J4.S
- new net AGND_KICK: A1.8 (AGND), J2.S
- new net AGND_SNARE: A1.10 (AGND), J3.S
- new net AGND_TOMS: A2.10 (AGND), J5.S
- new net COMPRESSOR_OUT: R78.2, SW26.2 (B), U10.7, U13.12 (+)
- new net HPFSTAGE_OUT: R59.1, SW26.5 (B), SW27.2 (B)
- new net HPF_IN: C74.1, SW26.3 (C)
- new net HPF_OUT: C76.2, R56.1, SW26.6 (C)
- new net LPFSTAGE_OUT: C3.2, R74.1, SW27.5 (B)
- new net LPF_IN: C78.1, SW27.3 (C)
- new net LPF_OUT: C81.2, R73.1, SW27.6 (C)
- new net MIXER_OUT: R46.2, R75.1, U2.7
Other:
- note added: "ANALOGUE SECTION"
- note added: "COMPRESSOR STAGE"
- note added: "CUT-OFF DUAL POT"
- note added: "DRIVE"
- note added: "DRUM VOICE BUFFERED OUTPUTS"
- note added: "FILTER STAGE"
- note added: "HPF SEMI-RESONANT"
- note added: "LEVEL POTS"
- note added: "LPF W/ RESONANCE"
- note added: "MASTER OUTPUT STAGE"
- note added: "MASTER VOLUME"
- note added: "MORITZ KLEIN COMPRESSOR"
- note added: "MORITZ KLEIN HPF"
- note added: "MORITZ KLEIN LPF"
- note added: "POWER SECTION"
- note added: "RATIO"
- note added: "RELEASE"
- note added: "RESONANCE"
- note added: "RESONANCE TRIM POT"
- note added: "SOFT CLIP STAGE"
- note added: "THRESHOLD"
- note added: "VIRTUAL RAILS"
- note removed: "ANALOGUE OUTPUT"
- note removed: "KICK DRUM FILTER STAGE"
- moved on the sheet: C1, C2, C69, C70, C71, C72, C73, Ch1, Ch2, Ch3, Ch4, D54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

Commit message: V0.3
Parts:
- A1, A2: footprint (none) -> PCM5102_DAC_BreakoutBoard_v2:PCM5102_DAC_BreakoutBoard
- D1: footprint (none) -> DIYSynthMNL:D_4148_BigPads
- D10, D11, D12, D13, D14, D15, D16, D17, D18, D19, D20, D21, D22, D23, D24, D25, D26, D27, D28, D29, D5, D6, D7, D8, D9: footprint (none) -> PCM_4ms_Diode:D_DO-35_P7.62mm_Horizontal
- D63, D64, D65, D66: footprint Diode_THT:D_DO-35_SOD27_P5.08mm_Vertical_KathodeUp -> PCM_4ms_Diode:D_DO-35_P7.62mm_Horizontal
- J6, TRS_JACK_1, TRS_JACK_2, TRS_JACK_3: footprint (none) -> audioConnectors_Edit:Jack_3.5mm_CUI_SJ1-3525N_Horizontal_edit
- R10, R11, R38, R39, R40, R41, R42, R43, R44, R45, R46, R47, R48, R49, R50, R51, R53, R54, R55, R56, R57, R58, R59, R60, R61, R62, R63, R64, R7, R70, R71, R72, R73, R74, R75, R76, R77, R78, R79, R8, R80, R81, R82, R83, R84, R85, R86, R87, R88, R9, R91, R92, R93, R94, R95, R96, R97, R98, R99: footprint (none) -> PCM_4ms_Resistor:R_Axial_DIN0207_L6.3mm_D2.5mm_P7.62mm_Horizontal
- R52: value 1k -> 2k; footprint (none) -> PCM_4ms_Resistor:R_Axial_DIN0207_L6.3mm_D2.5mm_P7.62mm_Horizontal
- RV1, RV10, RV11, RV12, RV13, RV14, RV15, RV16, RV17, RV18, RV19, RV2, RV20, RV21, RV22, RV23, RV24, RV25, RV26, RV3, RV4, RV5, RV6, RV7, RV8, RV9: footprint PCM_4ms_Potentiometer:Pot_9mm_Knurl_NoDet -> DIYSynthMNL:Potentiometer_RV09_BigPads
- RV27, RV28: footprint (none) -> PCM_4ms_Potentiometer:Potentiometer_Alps_RK09L_Double_Vertical
- RV33: renamed from Ch3; footprint (none) -> DIYSynthMNL:Potentiometer_RV09_BigPads
- RV35: renamed from Ch4; footprint (none) -> DIYSynthMNL:Potentiometer_RV09_BigPads
- RV37: renamed from RV1; footprint PCM_4ms_Potentiometer:Pot_9mm_Knurl_NoDet -> DIYSynthMNL:Potentiometer_RV09_BigPads
- RV38: renamed from Ch5; footprint (none) -> DIYSynthMNL:Potentiometer_RV09_BigPads
- RV39: renamed from Ch6; footprint (none) -> DIYSynthMNL:Potentiometer_RV09_BigPads
- RV40: renamed from Ch2; footprint (none) -> DIYSynthMNL:Potentiometer_RV09_BigPads
- RV46: renamed from Ch1; footprint (none) -> DIYSynthMNL:Potentiometer_RV09_BigPads
- SW1, SW10, SW11, SW12, SW13, SW14, SW15, SW16, SW17, SW18, SW19, SW2, SW20, SW21, SW22, SW23, SW24, SW25, SW3, SW4, SW5, SW6, SW7, SW8, SW9: footprint (none) -> PCM_Switch_Keyboard_Cherry_MX:SW_Cherry_MX_PCB_1.00u
- Teensy4.0: footprint (none) -> teensy:Teensy40
- U10, U12, U2, U3: footprint 4ms_Package_SSOP:TSSOP-8_4.4x3mm_Pitch0.65mm -> DIYSynthMNL:DIP-8_W7.62mm_LongPads
- U13, U14, U4: footprint (none) -> DIYSynthMNL:DIP-14_W7.62mm_LongPads
- U2, U3: footprint Package_DIP:DIP-8_W7.62mm -> DIYSynthMNL:DIP-8_W7.62mm_LongPads
- renumbered Nano to Nano1
Connections:
- net HATSBUFFER_IN: now also RV33.3; no longer RV33.2
- net HATS_OUT: now also RV33.2; no longer RV33.3
- net KICKBUFFER_IN: now also RV46.3; no longer RV46.2
- net KICK_OUT: now also RV46.2; no longer RV46.3
- net SNAREBUFFER_IN: now also RV40.3; no longer RV40.2
- net SNARE_OUT: now also RV40.2; no longer RV40.3
- net TOMSBUFFER_IN: now also RV35.3; no longer RV35.2
- net TOMS_OUT: now also RV35.2; no longer RV35.3
Other:
- moved on the sheet: U3C

Commit message: v0.4.0
- Modified mixer stage. Passive attenuators before DC bias to use the Differential Amplifier as a mixer.
Parts:
- added C4, C5, C6: 10uF, Capacitor_THT:CP_Radial_D5.0mm_P2.00mm, symbol Device:C_Polarized_US
- added R1, R2, R3, R4, R5, R6: 10k, PCM_4ms_Resistor:R_Axial_DIN0207_L6.3mm_D2.5mm_P7.62mm_Horizontal, symbol Device:R
- added R12: 22k, PCM_4ms_Resistor:R_Axial_DIN0207_L6.3mm_D2.5mm_P7.62mm_Horizontal, symbol Device:R
- added TRIM3: TrimPot_T73YEt_100k, DIYSynthMNL:Potentiometer_Bourns_3296W_Vertical_BigPads, symbol PCM_4ms_Potentiometer:TrimPot_T73YEt_100k
- added U15, U16: TL072, 4ms_Package_SSOP:TSSOP-8_4.4x3mm_Pitch0.65mm, symbol PCM_4ms_IC:TL072
Connections:
- net 5v is gone; now on net 12V: R42.2, R47.2
- net 12V: now also R1.2, R3.2, R5.2, U15.8 (V+)
- net COMPRESSOR_OUT: now also RV32.2, RV32.3, U16.1; no longer R78.2, U10.7, U13.12 (+)
- net GND: now also R2.1, R4.1, R6.1, U15.4 (V-)
- net HATSBUFFER_IN: now also C5.2; no longer R40.1
- net KICKBUFFER_IN: now also C3.2; no longer R38.1
- net LPFSTAGE_OUT: now also U3.3 (+); no longer C3.2
- net SNAREBUFFER_IN: no longer R39.1
- net TOMSBUFFER_IN: now also C6.2; no longer R41.1
- net VGND: now also R12.1
- net at C82.2, R86.1, TRIM2.1 (Left)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: now also TRIM3.3 (Right); no longer RV32.3
- net KICK_DCBIAS_OUT: now reaches C3.1, R49.1, R50.2
- net KICK_DCBIAS_OUT: now also R38.1; no longer U3.3 (+)
- new net: R78.2, U10.7, U13.12 (+), U16.3 (+)
- new net: R89.2, TRIM3.1 (Left), TRIM3.2 (Center)
- new net: R12.2, RV32.1, U16.2 (-)
- new net HATS_DCBIAS_OUT: C5.1, R3.1, R4.2, R40.1
- new net SNARE_DCBIAS_OUT: C4.1, R1.1, R2.2, R39.1
- new net TOMS_DCBIAS_OUT: C6.1, R41.1, R5.1, R6.2
Other:
- note added: "DC BIASING"
- note added: "DIFFERENTIAL MIXER"
- note added: "PASSIVE ATTENUATORS"
- moved on the sheet: C3, C82, C83, D3, D4, D55, D56, D57, D58, D59, D60, D61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
