File: build/FM_DRUM_MACHINE/FM_DRUM_MACHINE.kicad_pcb (KiCad board)
At the start: 2 copper layers, 510 x 257 mm, 273 parts, among them J1 12V Centre +ve, J2 KICK_BUFFEREDOUT, J3 SNARE_BUFFEREDOUT, J4 HATS_BUFFEREDOUT, J5 TOMS_BUFFEREDOUT, J6 LINE_OUT, Q1 BC547, Q2 BC557, SW1 STEP1, SW10 STEP10, SW11 STEP11, SW12 STEP12, SW13 STEP13, SW14 STEP14, SW15 STEP15, SW16 STEP16, SW17 KICK_TRIG, SW18 SNARE_TRIG, SW19 CHAT_TRIG, SW2 STEP2, SW20 OHAT_TRIG, SW21 LOTOM_TRIG, SW22 HITOM_TRIG, SW23 PLAY/PAUSE, SW24 RECORD, SW25 SELECT, SW26 SW_DPDT_x2, SW27 SW_DPDT_x2, SW3 STEP3, SW4 STEP4, SW5 STEP5, SW6 STEP6, SW7 STEP7, SW8 STEP8, SW9 STEP9, U1 6N138, U10 TL072, U11 TL074, U12 TL072, U13 TL074, U14 TL074, U2 TL072, U3 TL072, U4 TL074, U5 MAX7221xNG, U6 CD74HC4067M, U7 CD74HC4067M, U8 AMS1117-5.0, U9 AMS1117-3.3

Commit message: v0.5
POWER IN BOARD
Parts:
- added C4: 10uF, Capacitor_THT:CP_Radial_D5.0mm_P2.00mm, F.Cu at (-42.3, 220.9)
- added C5: 10uF, Capacitor_THT:CP_Radial_D5.0mm_P2.00mm, F.Cu at (-42.3, 227.4)
- added C6: 10uF, Capacitor_THT:CP_Radial_D5.0mm_P2.00mm, F.Cu at (-42.3, 234.0)
- added R1: 10k, PCM_4ms_Resistor:R_Axial_DIN0207_L6.3mm_D2.5mm_P7.62mm_Horizontal, F.Cu at (-49.9, 219.4)
- added R12: 22k, PCM_4ms_Resistor:R_Axial_DIN0207_L6.3mm_D2.5mm_P7.62mm_Horizontal, F.Cu at (-49.9, 240.7)
- added R2: 10k, PCM_4ms_Resistor:R_Axial_DIN0207_L6.3mm_D2.5mm_P7.62mm_Horizontal, F.Cu at (-49.9, 222.9)
- added R3: 10k, PCM_4ms_Resistor:R_Axial_DIN0207_L6.3mm_D2.5mm_P7.62mm_Horizontal, F.Cu at (-49.9, 226.5)
- added R4: 10k, PCM_4ms_Resistor:R_Axial_DIN0207_L6.3mm_D2.5mm_P7.62mm_Horizontal, F.Cu at (-49.9, 230.1)
- added R5: 10k, PCM_4ms_Resistor:R_Axial_DIN0207_L6.3mm_D2.5mm_P7.62mm_Horizontal, F.Cu at (-49.9, 233.6)
- added R6: 10k, PCM_4ms_Resistor:R_Axial_DIN0207_L6.3mm_D2.5mm_P7.62mm_Horizontal, F.Cu at (-49.9, 237.2)
- added R65: 10k, PCM_4ms_Resistor:R_Axial_DIN0207_L6.3mm_D2.5mm_P7.62mm_Horizontal, F.Cu at (-206.2, 156.8)
- added R66: 10k, PCM_4ms_Resistor:R_Axial_DIN0207_L6.3mm_D2.5mm_P7.62mm_Horizontal, F.Cu at (-206.2, 160.3)
- added R67: 10k, PCM_4ms_Resistor:R_Axial_DIN0207_L6.3mm_D2.5mm_P7.62mm_Horizontal, F.Cu at (-206.2, 163.9)
- added R68: 10k, PCM_4ms_Resistor:R_Axial_DIN0207_L6.3mm_D2.5mm_P7.62mm_Horizontal, F.Cu at (-206.2, 167.4)
- added R69: 10k, PCM_4ms_Resistor:R_Axial_DIN0207_L6.3mm_D2.5mm_P7.62mm_Horizontal, F.Cu at (-206.2, 171.0)
- added R89: 4k7, PCM_4ms_Resistor:R_Axial_DIN0207_L6.3mm_D2.5mm_P7.62mm_Horizontal, F.Cu at (-50.2, 246.5)
- added TRIM3: TrimPot_T73YEt_100k, DIYSynthMNL:Potentiometer_Bourns_3296W_Vertical_BigPads, F.Cu at (-36.5, 240.5)
- added U15: TL072, DIYSynthMNL:DIP-8_W7.62mm_LongPads, F.Cu at (-50.5, 260.9)
- J1: value 12V Centre +ve -> PJ-102A; footprint Connector_BarrelJack:BarrelJack_SwitchcraftConxall_RAPC10U_Horizontal -> PJ-102A:CUI_PJ-102A
- moved RV39 644.2 mm to (449.0, 52.8), turned to -90 degrees
- moved RV32 595.6 mm to (404.7, 53.0), turned to -90 degrees
- moved RV2 586.8 mm to (449.0, 114.1), turned to -90 degrees
- moved RV30 571.2 mm to (384.0, 52.8), turned to -90 degrees
- moved RV29 560.0 mm to (376.8, 114.3), turned to -90 degrees
- moved RV31 552.6 mm to (363.3, 52.8), turned to -90 degrees
- moved RV38 547.6 mm to (364.3, 145.3), turned to -90 degrees
- moved Teensy4.0 543.9 mm to (376.3, -116.4), turned to -90 degrees
- moved RV35 534.5 mm to (306.5, 89.3), turned to -90 degrees
- moved Nano1 531.5 mm to (389.1, -24.6), turned to -90 degrees
- moved SW26 520.9 mm to (374.2, 92.0)
- moved SW27 520.4 mm to (374.2, 104.0)
- moved RV37 512.2 mm to (449.0, 89.1), turned to -90 degrees
- moved RV22 467.4 mm to (319.0, 114.3), turned to -90 degrees
- moved RV33 458.8 mm to (229.0, 114.3), turned to -90 degrees
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Connections:
- C3 pad 1: Net-(U3A-+) -> KICK_DCBIAS_OUT
- C3 pad 2: LPFSTAGE_OUT -> KICKBUFFER_IN
- J1 pad 1: unconnected-(J1-Pad1) -> GND
- R38 pad 1: KICKBUFFER_IN -> KICK_DCBIAS_OUT
- R39 pad 1: SNAREBUFFER_IN -> SNARE_DCBIAS_OUT
- R40 pad 1: HATSBUFFER_IN -> HATS_DCBIAS_OUT
- R41 pad 1: TOMSBUFFER_IN -> TOMS_DCBIAS_OUT
- R42 pad 2: 5v -> 12V
- R47 pad 2: 5v -> 12V
- R49 pad 1: Net-(U3A-+) -> KICK_DCBIAS_OUT
- R50 pad 2: Net-(U3A-+) -> KICK_DCBIAS_OUT
- R78 pad 2: COMPRESSOR_OUT -> Net-(U13D-+)
- RV32 pad 1: Net-(R89-Pad2) -> Net-(U16A--)
- RV32 pad 2: Net-(R89-Pad2) -> COMPRESSOR_OUT
- RV32 pad 3: Net-(TRIM2-Center) -> COMPRESSOR_OUT
- U10 pad 7: COMPRESSOR_OUT -> Net-(U13D-+)
- U13 pad 12: COMPRESSOR_OUT -> Net-(U13D-+)
- U3 pad 3: Net-(U3A-+) -> LPFSTAGE_OUT
Other:
- board size 510 x 257 mm -> 417.9 x 188.1 mm

Commit message: v0.5.5
- Drive section modified based on testing
- LPF/HPF Based on testing
Parts:
- removed D55, D56: 1N4148, Diode_THT:D_DO-35_SOD27_P5.08mm_Vertical_KathodeUp
- removed R42, R43, R47, R48, R49: 10k, PCM_4ms_Resistor:R_Axial_DIN0207_L6.3mm_D2.5mm_P7.62mm_Horizontal
- added R13: 820R, PCM_4ms_Resistor:R_Axial_DIN0207_L6.3mm_D2.5mm_P7.62mm_Horizontal, F.Cu at (-98.2, 262.6)
- added R14: 330R, PCM_4ms_Resistor:R_Axial_DIN0207_L6.3mm_D2.5mm_P7.62mm_Horizontal, F.Cu at (-98.2, 266.1)
- added R15: 330R, PCM_4ms_Resistor:R_Axial_DIN0207_L6.3mm_D2.5mm_P7.62mm_Horizontal, F.Cu at (-98.2, 269.7)
- D3: value 1N4148 -> RED LED
- D4: value 1N4148 -> 1N4007
- R1, R3, R5: value 10k -> 820R
- R2, R4, R50, R6: value 10k -> 330R
- R52: value 2k -> 680R
- R53, R56, R60, R73: value 200k -> 220k
- R58, R64: value 6k8 -> 10k
- RV29: value R_Potentiometer -> 100k
- RV38: value 20k -> B20k
- RV39: value 1k -> A1k
- moved R1 58.2 mm to (-98.2, 251.9)
- moved R3 56.3 mm to (-98.2, 255.5)
- moved R5 54.6 mm to (-98.2, 259.1)
Connections:
- C3 pad 1: KICK_DCBIAS_OUT -> KICKBUFFER_IN
- C3 pad 2: KICKBUFFER_IN -> KICK_DCBIAS_IN
- C4 pad 1: SNARE_DCBIAS_OUT -> SNAREBUFFER_IN
- C5 pad 1: HATS_DCBIAS_OUT -> HATSBUFFER_IN
- C5 pad 2: HATSBUFFER_IN -> HATS_DCBIAS_IN
- C6 pad 1: TOMS_DCBIAS_OUT -> TOMSBUFFER_IN
- C6 pad 2: TOMSBUFFER_IN -> TOMS_DCBIAS_IN
- D3 pad 2: Net-(D3-A) -> SOFTCLIP_OUT
- D4 pad 1: Net-(D3-A) -> SOFTCLIP_OUT
- D4 pad 2: SOFTCLIP_OUT -> Net-(D3-K)
- R1 pad 1: SNARE_DCBIAS_OUT -> Net-(U4A--)
- R1 pad 2: 12V -> Net-(R1-Pad2)
- R2 pad 1: GND -> VGND
- R2 pad 2: SNARE_DCBIAS_OUT -> SNAREBUFFER_IN
- R3 pad 1: HATS_DCBIAS_OUT -> Net-(U4B--)
- R3 pad 2: 12V -> Net-(U4B--)
- R38 pad 1: KICK_DCBIAS_OUT -> KICKBUFFER_IN
- R39 pad 1: SNARE_DCBIAS_OUT -> SNAREBUFFER_IN
- R4 pad 1: GND -> VGND
- R4 pad 2: HATS_DCBIAS_OUT -> HATSBUFFER_IN
- R40 pad 1: HATS_DCBIAS_OUT -> HATSBUFFER_IN
- R41 pad 1: TOMS_DCBIAS_OUT -> TOMSBUFFER_IN
- R5 pad 1: TOMS_DCBIAS_OUT -> Net-(R5-Pad1)
- R5 pad 2: 12V -> VGND
- R50 pad 1: GND -> VGND
- R50 pad 2: KICK_DCBIAS_OUT -> KICKBUFFER_IN
- R52 pad 1: VGND -> Net-(R52-Pad1)
- R52 pad 2: Net-(R52-Pad2) -> Net-(D3-K)
- R6 pad 1: GND -> VGND
- R6 pad 2: TOMS_DCBIAS_OUT -> TOMSBUFFER_IN
- RV27 pad 1: VGND -> Net-(R5-Pad1)
- RV28 pad 1: Net-(U4A--) -> Net-(R1-Pad2)
- RV29 pad 1: VGND -> Net-(R14-Pad2)
- RV33 pad 3: HATSBUFFER_IN -> HATS_DCBIAS_IN
- RV35 pad 3: TOMSBUFFER_IN -> TOMS_DCBIAS_IN
- RV38 pad 1: Net-(R52-Pad2) -> Net-(R52-Pad1)
- RV38 pad 2: Net-(R52-Pad2) -> Net-(R52-Pad1)
- RV38 pad 3: Net-(D3-K) -> VGND
- RV40 pad 3: SNAREBUFFER_IN -> SNARE_DCBIAS_IN
- RV46 pad 3: KICKBUFFER_IN -> KICK_DCBIAS_IN
- TRIM1 pad 1: VGND -> Net-(TRIM1-Left)
- U2 pad 3: Net-(U2A-+) -> VGND
- U2 pad 5: Net-(U2B-+) -> VGND

Commit message: PCB Changes
Parts:
- removed RV23: OHAT_DECAY, DIYSynthMNL:Potentiometer_RV09_BigPads
- removed RV24: OHAT_TIMBRE, DIYSynthMNL:Potentiometer_RV09_BigPads
- removed RV25: OHAT_PITCH, DIYSynthMNL:Potentiometer_RV09_BigPads
- removed RV26: OHAT_FMFREQ, DIYSynthMNL:Potentiometer_RV09_BigPads
- removed U12, U15: TL072, DIYSynthMNL:DIP-8_W7.62mm_LongPads
- added C7: 100uF, Capacitor_THT:CP_Radial_D5.0mm_P2.00mm, F.Cu at (103.5, 24.0)
- added R16: 10R, PCM_4ms_Resistor:R_Axial_DIN0207_L6.3mm_D2.5mm_P7.62mm_Horizontal, F.Cu at (96.3, 24.0)
- ATTACK: renamed from TRIM2; value TrimPot_T73YEt_100k -> 100k
- D3: footprint Diode_THT:D_DO-35_SOD27_P5.08mm_Vertical_KathodeUp -> LED_THT:LED_D5.0mm
- D4: value 1N4007 -> RED LED; footprint Diode_THT:D_DO-35_SOD27_P5.08mm_Vertical_KathodeUp -> LED_THT:LED_D5.0mm
- R88: value 20k -> 33k
- RELEASE: renamed from TRIM3; value TrimPot_T73YEt_100k -> 100k
- RV10: value SNARE_TIMBRE -> SNARE_TONE
- RV11: value CHAT_DECAY -> HAT_DECAY
- RV12: value CHAT_TIMBRE -> HAT_TIMBRE
- RV13: value CHAT_PITCH -> HAT_TONE
- RV14: value CHAT_FMFREQ -> HAT_RESONANCE
- RV17: value LOTOM_PITCH -> LOTOM_TUNE
- RV18: value LOTOM_FMFREQ -> LOTOM_ATTACK
- RV21: value HITOM_PITCH -> HITOM_TUNE
- RV22: value HITOM_FMFREQ -> HITOM_ATTACK
- RV3: value KICK_PITCH -> KICK_TUNE
- RV31: value 20k -> 10k
- RV5: value KICK_FMFREQ -> KICK_ATTACK
- RV9: value SNARE_FM -> SNARE_SNAP
- U10: value TL072 -> TL074; footprint DIYSynthMNL:DIP-8_W7.62mm_LongPads -> DIYSynthMNL:DIP-14_W7.62mm_LongPads
- U2, U3: footprint DIYSynthMNL:DIP-8_W7.62mm_LongPads -> Package_DIP:DIP-8_W7.62mm_LongPads
- moved R91 610.6 mm to (472.3, 35.5)
- moved R51 590.4 mm to (436.2, 103.5)
- moved U10 582.2 mm to (346.7, 47.2)
- moved R52 579.2 mm to (424.8, 96.9), turned to 90 degrees
- moved R83 543.7 mm to (391.1, 48.7), turned to -90 degrees
- moved C83 543.7 mm to (471.0, 48.5)
- moved R88 542.6 mm to (405.2, 42.8)
- moved R82 530.8 mm to (383.1, 78.0)
- moved J6 524.2 mm to (473.5, 24.5), turned to 180 degrees
- moved U13 522.5 mm to (368.8, 62.7)
- moved R79 512.4 mm to (361.3, 45.9), turned to -90 degrees
- moved R85 512.0 mm to (362.2, 75.5)
- moved R84 511.0 mm to (362.2, 78.2)
- moved R78 507.6 mm to (358.3, 53.4), turned to -90 degrees
- moved R87 504.2 mm to (367.3, 46.0), turned to -90 degrees
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Connections:
- net CHAT_DECAY renamed HAT_DECAY
- net CHAT_FMFREQ renamed HAT_RESONANCE
- net CHAT_PITCH renamed HAT_TONE
- net CHAT_TIMBRE renamed HAT_TIMBRE
- net KICK_FMFREQ renamed KICK_ATTACK
- net KICK_PITCH renamed KICK_TUNE
- net SNARE_FM renamed SNARE_SNAP
- net SNARE_TIMBRE renamed SNARE_TONE
- A1 pad 10: AGND_SNARE -> AGND
- A1 pad 12: GND -> DGND
- A1 pad 14: GND -> DGND
- A1 pad 15: GND -> DGND
- A1 pad 5: GND -> DGND
- A1 pad 8: AGND_KICK -> AGND
- A2 pad 10: AGND_TOMS -> AGND
- A2 pad 12: GND -> DGND
- A2 pad 14: GND -> DGND
- A2 pad 15: GND -> DGND
- A2 pad 5: GND -> DGND
- A2 pad 8: AGND_HATS -> AGND
- C1 pad 1: 12V -> A12V
- C2 pad 2: GND -> DGND
- C27 pad 1: Net-(C27-Pad1) -> TEMPO
- C27 pad 2: GND -> DGND
- C43 pad 1: Net-(C43-Pad1) -> SWING
- C43 pad 2: GND -> DGND
- C44 pad 2: GND -> DGND
- C45 pad 2: GND -> DGND
- C46 pad 2: GND -> DGND
- C47 pad 2: GND -> DGND
- C48 pad 2: GND -> DGND
- C49 pad 2: GND -> DGND
- C50 pad 2: GND -> DGND
- C51 pad 2: GND -> DGND
- C52 pad 2: GND -> DGND
- C53 pad 2: GND -> DGND
- C54 pad 2: GND -> DGND
- C55 pad 2: GND -> DGND
- C56 pad 2: GND -> DGND
- C57 pad 2: GND -> DGND
- C58 pad 2: GND -> DGND
- C59 pad 1: LOTOM_PITCH -> LOTOM_TUNE
- C59 pad 2: GND -> DGND
- C60 pad 1: LOTOM_FMFREQ -> LOTOM_ATTACK
- C60 pad 2: GND -> DGND
- C61 pad 2: GND -> DGND
- C62 pad 2: GND -> DGND
- C63 pad 2: GND -> DGND
- C64 pad 1: HITOM_FMFREQ -> HITOM_ATTACK
- C64 pad 2: GND -> DGND
- C69 pad 1: GND -> DGND
- C70 pad 1: GND -> DGND
- C71 pad 1: GND -> DGND
- C72 pad 1: GND -> DGND
- C73 pad 1: GND -> DGND
- C73 pad 2: Net-(U10A-+) -> Net-(U3A-+)
- C75 pad 1: Net-(U11A--) -> Net-(U4A--)
- C75 pad 2: Net-(U11C-+) -> Net-(U4C-+)
- C77 pad 2: Net-(U11B-+) -> Net-(U4B-+)
- C79 pad 2: Net-(U4B-+) -> Net-(U11B-+)
- C80 pad 1: VGND -> Vref
- C80 pad 2: Net-(U4C-+) -> Net-(U11C-+)
- C81 pad 1: Net-(U4C--) -> Net-(U11C--)
- C82 pad 1: VGND -> Vref
- J1 pad 1: GND -> DGND
- J2 pad S: AGND_KICK -> AGND
- J3 pad S: AGND_SNARE -> AGND
- J4 pad S: AGND_HATS -> AGND
- J5 pad S: AGND_TOMS -> AGND
- J6 pad S: GND -> AGND
- Nano1 pad 19: unconnected-(Nano1-A0-Pad19) -> X0
- Nano1 pad 20: unconnected-(Nano1-A1-Pad20) -> X1
- Nano1 pad 21: unconnected-(Nano1-A2-Pad21) -> X2
- Nano1 pad 22: unconnected-(Nano1-A3-Pad22) -> X3
- Nano1 pad 23: unconnected-(Nano1-A4-Pad23) -> X4
- Nano1 pad 24: unconnected-(Nano1-A5-Pad24) -> TEMPO
- Nano1 pad 25: unconnected-(Nano1-A6-Pad25) -> SWING
- Nano1 pad 29: GND -> DGND
- Nano1 pad 4: GND -> DGND
- Q1 pad 1: 12V -> A12V
- Q2 pad 1: GND -> DGND
- R1 pad 1: Net-(U4A--) -> Net-(U11A--)
- R12 pad 1: VGND -> Vref
- R12 pad 2: Net-(U16A--) -> Net-(U10C--)
- R13 pad 1: Net-(U11B--) -> Net-(U4B--)
- R13 pad 2: Net-(U11B--) -> Net-(U4B--)
- R14 pad 1: VGND -> Vref
- R15 pad 1: VGND -> Vref
- R2 pad 1: VGND -> Vref
- R3 pad 1: Net-(U4B--) -> Net-(U11B--)
- R3 pad 2: Net-(U4B--) -> Net-(U11B--)
- R38 pad 2: Net-(U2A--) -> Net-(U2B--)
- R39 pad 2: Net-(U2A--) -> Net-(U2B--)
- R4 pad 1: VGND -> Vref
- R40 pad 2: Net-(U2A--) -> Net-(U2B--)
- R41 pad 2: Net-(U2A--) -> Net-(U2B--)
- R44 pad 1: Net-(U2A--) -> Net-(U2B--)
- R45 pad 2: Net-(U2B--) -> Net-(U2A--)
- R46 pad 1: Net-(U2B--) -> Net-(U2A--)
- R5 pad 2: VGND -> Vref
- R50 pad 1: VGND -> Vref
- R53 pad 2: VGND -> Vref
- R54 pad 2: Net-(U11A-+) -> Net-(U4A-+)
- R55 pad 1: VGND -> Vref
- R55 pad 2: Net-(U11A-+) -> Net-(U4A-+)
- R56 pad 2: VGND -> Vref
- R57 pad 2: Net-(U11D--) -> Net-(U4D--)
- R58 pad 1: Net-(U11D--) -> Net-(U4D--)
- R58 pad 2: VGND -> Vref
- R59 pad 2: VGND -> Vref
- R6 pad 1: VGND -> Vref
- R60 pad 2: VGND -> Vref
- R61 pad 2: Net-(U4A-+) -> Net-(U11A-+)
- R62 pad 1: VGND -> Vref
- R62 pad 2: Net-(U4A-+) -> Net-(U11A-+)
- R63 pad 2: Net-(U4D--) -> Net-(U11D--)
- R64 pad 1: Net-(U4D--) -> Net-(U11D--)
- R64 pad 2: VGND -> Vref
- R65 pad 1: GND -> DGND
- R66 pad 1: GND -> DGND
- R67 pad 1: GND -> DGND
- R68 pad 1: GND -> DGND
- R69 pad 1: GND -> DGND
- R7 pad 1: GND -> DGND
- R70 pad 1: 12V -> A12V
- R70 pad 2: Net-(U10A-+) -> Net-(U3A-+)
- R71 pad 1: Net-(U10A-+) -> Net-(U3A-+)
- R71 pad 2: GND -> DGND
- R73 pad 2: VGND -> Vref
- R74 pad 2: VGND -> Vref
- R75 pad 2: Net-(U12A-+) -> Net-(U10A-+)
- R76 pad 1: VGND -> Vref
- R76 pad 2: Net-(U12A-+) -> Net-(U10A-+)
- R77 pad 1: Net-(U12A--) -> Net-(U10A--)
- R78 pad 1: Net-(U10B--) -> Net-(U10D--)
- R78 pad 2: Net-(U13D-+) -> Net-(U10C-+)
- R79 pad 1: VGND -> Vref
- R79 pad 2: Net-(U10B--) -> Net-(U10D--)
- R80 pad 1: Net-(U13A--) -> Net-(U10B--)
- R81 pad 2: Net-(U13A--) -> Net-(U10B--)
- R83 pad 1: VGND -> Vref
- R84 pad 1: Net-(U13C--) -> Net-(U13B--)
- R85 pad 2: Net-(U13C--) -> Net-(U13B--)
- R86 pad 2: Net-(U13C-+) -> Net-(U13B-+)
- R87 pad 1: VGND -> Vref
- R87 pad 2: Net-(U13C-+) -> Net-(U13B-+)
- R88 pad 1: 12V -> A12V
- R89 pad 1: VGND -> Vref
- R96 pad 2: GND -> AGND
- R97 pad 2: GND -> AGND
- R98 pad 2: GND -> unconnected-(R98-Pad2)
- R99 pad 2: GND -> AGND
- RV1 pad 1: GND -> DGND
- RV10 pad 1: GND -> DGND
- RV11 pad 1: GND -> DGND
- RV12 pad 1: GND -> DGND
- RV13 pad 1: GND -> DGND
- RV14 pad 1: GND -> DGND
- RV15 pad 1: GND -> DGND
- RV16 pad 1: GND -> DGND
- RV17 pad 1: GND -> DGND
- RV17 pad 2: LOTOM_PITCH -> LOTOM_TUNE
- RV18 pad 1: GND -> DGND
- RV18 pad 2: LOTOM_FMFREQ -> LOTOM_ATTACK
- RV19 pad 1: GND -> DGND
- RV2 pad 1: GND -> DGND
- RV2 pad 2: Net-(C43-Pad1) -> SWING
- RV20 pad 1: GND -> DGND
- RV21 pad 1: GND -> DGND
- RV22 pad 1: GND -> DGND
- RV22 pad 2: HITOM_FMFREQ -> HITOM_ATTACK
- RV27 pad 2: Net-(U11B-+) -> Net-(U4B-+)
- RV27 pad 3: Net-(U11B-+) -> Net-(U4B-+)
- RV27 pad 4: Net-(U11B--) -> Net-(U4B--)
- RV27 pad 5: Net-(U11C-+) -> Net-(U4C-+)
- RV27 pad 6: Net-(U11C-+) -> Net-(U4C-+)
- RV28 pad 2: Net-(U4B-+) -> Net-(U11B-+)
- RV28 pad 3: Net-(U4B-+) -> Net-(U11B-+)
- RV28 pad 4: Net-(U4B--) -> Net-(U11B--)
- RV28 pad 5: Net-(U4C-+) -> Net-(U11C-+)
- RV28 pad 6: Net-(U4C-+) -> Net-(U11C-+)
- RV29 pad 2: Net-(U4D-+) -> Net-(U11D-+)
- RV29 pad 3: Net-(U4C--) -> Net-(U11C--)
- RV3 pad 1: GND -> DGND
- RV30 pad 2: Net-(U13B-+) -> Net-(U13C-+)
- RV30 pad 3: VGND -> Vref
- RV31 pad 1: VGND -> Vref
- RV32 pad 1: Net-(U16A--) -> Net-(U10C--)
- RV33 pad 1: GND -> AGND
- RV35 pad 1: GND -> AGND
- RV37 pad 1: GND -> DGND
- RV37 pad 2: Net-(C27-Pad1) -> TEMPO
- RV38 pad 3: VGND -> Vref
- RV39 pad 1: GND -> AGND
- RV4 pad 1: GND -> DGND
- RV40 pad 1: GND -> AGND
- RV46 pad 1: GND -> AGND
- RV5 pad 1: GND -> DGND
- RV6 pad 1: GND -> DGND
- RV7 pad 1: GND -> DGND
- RV8 pad 1: GND -> DGND
- RV9 pad 1: GND -> DGND
- TRS_JACK_1 pad S: GND -> DGND
- TRS_JACK_2 pad S: GND -> DGND
- TRS_JACK_3 pad S: GND -> DGND
- Teensy4.0 pad 1: GND -> DGND
- Teensy4.0 pad 32: GND -> DGND
- U1 pad 5: GND -> DGND
- U10 pad 1: Net-(Q1-B) -> Net-(U10A--)
- U10 pad 2: Net-(Q1-E) -> Net-(U10A--)
- U10 pad 4: GND -> A12V
- U10 pad 5: Net-(D57-K) -> Vref
- U10 pad 7: Net-(U13D-+) -> Net-(D62-K)
- U10 pad 8: 12V -> COMPRESSOR_OUT
- U11 pad 11: GND -> AGND
- U11 pad 12: Net-(TRIM1-Center) -> Net-(U11D-+)
- U11 pad 14: Net-(C77-Pad1) -> Net-(C79-Pad1)
- U11 pad 4: 12V -> A12V
- U11 pad 8: Net-(TRIM1-Right) -> Net-(U11C--)
- U11 pad 9: Net-(TRIM1-Right) -> Net-(U11C--)
- U13 pad 1: Net-(D62-K) -> Net-(D67-A)
- U13 pad 11: GND -> AGND
- U13 pad 12: Net-(U13D-+) -> LPFSTAGE_OUT
- U13 pad 13: Net-(TRIM2-Center) -> Net-(D3-K)
- U13 pad 14: Net-(D67-A) -> SOFTCLIP_OUT
- U13 pad 2: Net-(U13A--) -> Net-(TRIM2-Center)
- U13 pad 3: VGND -> Net-(U10C-+)
- U13 pad 4: 12V -> A12V
- U13 pad 6: Net-(D63-K) -> Net-(U13B--)
- U13 pad 7: Net-(R82-Pad1) -> Net-(R84-Pad2)
- U13 pad 8: Net-(R84-Pad2) -> Net-(R82-Pad1)
- U13 pad 9: Net-(U13C--) -> Net-(D63-K)
- U14 pad 11: GND -> AGND
- U14 pad 4: 12V -> A12V
- U2 pad 1: Net-(R44-Pad2) -> MIXER_OUT
- U2 pad 3: VGND -> Vref
- U2 pad 4: GND -> AGND
- U2 pad 5: VGND -> Vref
- U2 pad 7: MIXER_OUT -> Net-(R44-Pad2)
- U2 pad 8: 12V -> A12V
- U3 pad 1: SOFTCLIP_OUT -> Net-(Q1-B)
- U3 pad 2: Net-(D3-K) -> Net-(Q1-E)
- U3 pad 3: LPFSTAGE_OUT -> Net-(U3A-+)
- U3 pad 4: GND -> DGND
- U3 pad 6: VGND -> Vref
- U3 pad 7: VGND -> Vref
- U3 pad 8: 12V -> A12V
- U4 pad 11: GND -> AGND
- U4 pad 12: Net-(U4D-+) -> Net-(TRIM1-Center)
- U4 pad 14: Net-(C79-Pad1) -> Net-(C77-Pad1)
- U4 pad 4: 12V -> A12V
- U4 pad 8: Net-(U4C--) -> Net-(TRIM1-Right)
- U4 pad 9: Net-(U4C--) -> Net-(TRIM1-Right)
- U5 pad 4: GND -> DGND
- U5 pad 9: GND -> DGND
- U6 pad 12: GND -> DGND
- U6 pad 15: GND -> DGND
- U6 pad 16: OHAT_TIMBRE -> unconnected-(U6-I15-Pad16)
- U6 pad 17: OHAT_PITCH -> unconnected-(U6-I14-Pad17)
- U6 pad 18: OHAT_DECAY -> unconnected-(U6-I13-Pad18)
- U7 pad 12: GND -> DGND
- U7 pad 15: GND -> DGND
- U7 pad 2: HITOM_PUNCH -> HITOM_ATTACK
- U7 pad 23: HITOM_FMFREQ -> unconnected-(U7-I8-Pad23)
- U7 pad 3: HITOM_PITCH -> HITOM_PUNCH
- U7 pad 4: HITOM_DECAY -> HITOM_PITCH
- U7 pad 5: LOTOM_FMFREQ -> HITOM_DECAY
- U7 pad 6: LOTOM_PUNCH -> LOTOM_ATTACK
- U7 pad 7: LOTOM_PITCH -> LOTOM_PUNCH
- U7 pad 8: LOTOM_DECAY -> LOTOM_TUNE
- U7 pad 9: OHAT_FMFREQ -> LOTOM_DECAY
- U8 pad 1: GND -> DGND
- U9 pad 1: GND -> DGND
Routing:
- net COMPRESSOR_OUT: track 0.00 -> 213.3 mm
- net Net-(D3-K): track 0.00 -> 147.8 mm, vias 0 -> 1
- net Net-(D59-A): track 0.00 -> 126.2 mm
- net Vref: track 0.00 -> 123.8 mm
- net SOFTCLIP_OUT: track 0.00 -> 112.8 mm, vias 0 -> 1
- net Net-(U10C--): track 0.00 -> 94.5 mm
- net Net-(R85-Pad1): track 0.00 -> 90.7 mm
- net Net-(TRIM2-Center): track 0.00 -> 70.0 mm
- net AGND: track 0.00 -> 68.8 mm
- net A12V: track 0.00 -> 68.2 mm
- net Net-(R84-Pad2): track 0.00 -> 56.5 mm
- net Net-(Q1-E): track 0.00 -> 44.4 mm
- net Net-(U10C-+): track 0.00 -> 42.6 mm
- net Net-(U13C-+): track 0.00 -> 40.8 mm
- net Net-(D62-K): track 0.00 -> 39.3 mm
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Other:
- board outline removed
- board text added: "COMPRESSOR"

Commit message: Schematic PCB Changes
- Updated Power In
- Updated PCB
Parts:
- removed C65, C66, C67, C68: 10nF, PCM_4ms_Capacitor:C_Disc_P5.08mm
- removed C7: 100uF, Capacitor_THT:CP_Radial_D5.0mm_P2.00mm
- removed Q1: BC547, Package_TO_SOT_THT:TO-92L_Inline
- removed Q2: BC557, Package_TO_SOT_THT:TO-92_Inline
- removed R16: 10R, PCM_4ms_Resistor:R_Axial_DIN0207_L6.3mm_D2.5mm_P7.62mm_Horizontal
- removed R72: 1k, PCM_4ms_Resistor:R_Axial_DIN0207_L6.3mm_D2.5mm_P7.62mm_Horizontal
- removed R96, R97, R98, R99: 220R, PCM_4ms_Resistor:R_Axial_DIN0207_L6.3mm_D2.5mm_P7.62mm_Horizontal
- added TRIM2: TrimPot_T73YEt_100k, DIYSynthMNL:Potentiometer_Bourns_3296W_Vertical_BigPads, F.Cu at (-120.6, 197.1)
- added TRIM3: TrimPot_T73YEt_100k, DIYSynthMNL:Potentiometer_Bourns_3296W_Vertical_BigPads, F.Cu at (-120.6, 203.5)
- added U12: OPA551P, Package_DIP:DIP-8_W7.62mm, F.Cu at (82.4, 69.5)
- D10, D11, D12, D13, D14, D15, D16, D17, D18, D19, D20, D21, D22, D23, D24, D25, D26, D27, D28, D29, D5, D6, D7, D8, D9: value Random Diode -> 1N4148
- R82: value 1k -> 2k
- U3: value TL072 -> OPA551P; footprint Package_DIP:DIP-8_W7.62mm_LongPads -> Package_DIP:DIP-8_W7.62mm
- moved D52 931.1 mm to (-437.1, 330.9)
- moved D51 915.2 mm to (-437.1, 323.5)
- moved D50 900.4 mm to (-437.1, 316.0)
- moved A2 857.8 mm to (-520.1, 103.7)
- moved A1 797.5 mm to (-536.8, 78.8)
- moved RV28 735.3 mm to (-223.5, 322.0)
- moved RV29 735.3 mm to (-196.0, 314.5)
- moved D53 733.7 mm to (-437.1, 338.4)
- moved ATTACK 707.1 mm to (621.5, -614.9)
- moved C82 707.1 mm to (614.8, -617.7)
- moved D3 707.1 mm to (654.9, -553.0)
- moved D4 707.1 mm to (677.3, -553.0)
- moved D57 707.1 mm to (587.3, -626.4)
- moved D58 707.1 mm to (589.8, -629.4)
- moved D59 707.1 mm to (595.3, -626.4)
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Connections:
- C1 pad 1: A12V -> 12V
- C1 pad 2: Net-(Q1-E) -> Net-(U12-+)
- C2 pad 1: Net-(Q1-E) -> Net-(U12-+)
- D65 pad 1: Net-(D64-A) -> Net-(D63-A)
- D65 pad 2: Net-(D59-A) -> Net-(D65-A)
- D66 pad 1: Net-(D59-A) -> Net-(D65-A)
- J2 pad S: AGND -> DGND
- J3 pad S: AGND -> DGND
- J4 pad S: AGND -> DGND
- J5 pad S: AGND -> DGND
- J6 pad S: AGND -> DGND
- R7 pad 1: DGND -> Net-(D1-K)
- R7 pad 2: Net-(D1-K) -> Net-(R7-Pad2)
- R70 pad 1: A12V -> 12V
- R82 pad 1: Net-(R82-Pad1) -> Net-(D65-A)
- R88 pad 1: A12V -> 12V
- RV33 pad 1: AGND -> DGND
- RV35 pad 1: AGND -> DGND
- RV39 pad 1: AGND -> DGND
- RV40 pad 1: AGND -> DGND
- RV46 pad 1: AGND -> DGND
- TRS_JACK_1 pad R: Net-(D1-A) -> Net-(R7-Pad2)
- TRS_JACK_1 pad T: Net-(TRS_JACK_1-PadT) -> Net-(D1-A)
- TRS_JACK_2 pad R: Net-(D1-A) -> Net-(R7-Pad2)
- TRS_JACK_2 pad T: Net-(TRS_JACK_1-PadT) -> Net-(D1-A)
- U10 pad 11: AGND -> DGND
- U10 pad 4: A12V -> 12V
- U11 pad 11: AGND -> DGND
- U11 pad 4: A12V -> 12V
- U13 pad 11: AGND -> DGND
- U13 pad 4: A12V -> 12V
- U13 pad 8: Net-(R82-Pad1) -> Net-(D65-A)
- U14 pad 11: AGND -> DGND
- U14 pad 4: A12V -> 12V
- U2 pad 4: AGND -> DGND
- U2 pad 8: A12V -> 12V
- U3 pad 1: Net-(Q1-B) -> unconnected-(U3-NC-Pad1)
- U3 pad 2: Net-(Q1-E) -> Net-(U12-+)
- U3 pad 5: Net-(Q1-E) -> unconnected-(U3-NC-Pad5)
- U3 pad 6: Vref -> Net-(U12-+)
- U3 pad 7: Vref -> 12V
- U3 pad 8: A12V -> DGND
- U4 pad 11: AGND -> DGND
- U4 pad 4: A12V -> 12V
Routing:
- net DIG0: track 0.00 -> 319.2 mm
- net DIG1: track 0.00 -> 224.1 mm
- net DIG2: track 0.00 -> 221.3 mm
- net DIG3: track 0.00 -> 220.7 mm
- net DIG4: track 0.00 -> 219.2 mm
- net 12V: track 28.3 -> 173.5 mm
- net SEGC: track 0.00 -> 90.2 mm
- net SEGA: track 0.00 -> 87.7 mm
- net SEGB: track 0.00 -> 87.5 mm
- net DGND: track 0.00 -> 82.6 mm
- net AGND: track 68.8 -> 0.00 mm
- net A12V: track 68.2 -> 0.00 mm
- net Net-(U14D--): track 0.00 -> 48.2 mm
- net Net-(U12-+): track 0.00 -> 45.1 mm
- net Net-(Q1-E): track 44.4 -> 0.00 mm
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Other:
- board text added: "DRUM VOICE OUTPUTS"
- board text added: "MIDI"
- board text added: "POWER"
